File: PCB/Fuente de tensión regulable.kicad_pcb (KiCad board)
At the start: 2 copper layers, 90 x 58 mm, 35 parts, among them J2 conector DC, J3 conector current, SW1 SW_Wuerth_450301014042, U1 L7805, U3 LM2596S-12

Commit message: Add files via upload
Parts:
- moved U1 3.70 mm to (170.3, 70.6), turned to -90 degrees
- moved C6 2.66 mm to (177.5, 67.4)
- moved C5 1.71 mm to (176.7, 72.3)
Routing:
- net 5v: track 58.6 -> 65.1 mm
- net /+: track 144.0 -> 150.2 mm

Commit message: Add files via upload
Parts:
- U1: value L7805 -> AMS1117-5.0
- moved U1 0.16 mm to (170.2, 70.8)
Connections:
- U1 pad 1: /+ -> GND
- U1 pad 2: GND -> 5v
- U1 pad 3: 5v -> /+

Commit message: Add files via upload
Parts:
- SW1: footprint Connector_PinHeader_2.54mm:PinHeader_1x03_P2.54mm_Vertical -> TerminalBlock:TerminalBlock_MaiXu_MX126-5.0-02P_1x02_P5.00mm
- moved SW1 0.25 mm to (210.5, 104.5), turned to 90 degrees
Connections:
- SW1 pad 3: Net-(SW1-A) -> unconnected-(SW1-C-Pad2)
Routing:
- net /+: track 150.4 -> 160.2 mm
- net 5v: track 65.2 -> 71.5 mm
